Commit message: Class for crawler robot, modified xacro
Xacro has been modified inverting the order of the joints connecting the girdle to the leg to simplify the position control of the flexion joint. Other minor modifications to the model structure.
crawler.py define the Crawler class and gathers all the functions related to the model.

File: crawler.urdf (robot description, URDF)
Before this commit: robot crawler, 21 links, 20 joints
Links:
- link girdle: mass 0.1 -> 0.111111111111; geometry collision sphere radius=0.0625; collision sphere radius=0.0625
- link left_girdle_connection_1: mass 0.01 -> 0.000111111111111
- link left_leg: mass 0.05 -> 0.0111111111111; geometry collision sphere radius=0.0208333333333; visual box size=0.125 0.0125 0.0125
- link right_girdle_connection_1: mass 0.01 -> 0.000111111111111
- link right_leg: mass 0.05 -> 0.0111111111111; geometry collision sphere radius=0.0208333333333; visual box size=0.125 0.0125 0.0125
- link spine_connection_1: mass 0.001 -> 0.00111111111111
- link spine_connection_2: mass 0.001 -> 0.00111111111111
- link spine_connection_3: mass 0.001 -> 0.00111111111111
- link spine_connection_4: mass 0.001 -> 0.00111111111111
- link spine_connection_5: mass 0.001 -> 0.00111111111111
- link spine_connection_6: mass 0.001 -> 0.00111111111111
- link spine_connection_7: mass 0.001 -> 0.00111111111111
- link spine_connection_8: mass 0.001 -> 0.00111111111111
- link spine_link_1: mass 0.1 -> 0.111111111111; geometry collision sphere radius=0.0625; visual box size=0.125 0.0125 0.00625
- link spine_link_2: mass 0.1 -> 0.111111111111; geometry collision sphere radius=0.0625; visual box size=0.125 0.0125 0.00625
- link spine_link_3: mass 0.1 -> 0.111111111111; geometry collision sphere radius=0.0625; visual box size=0.125 0.0125 0.00625
- link spine_link_4: mass 0.1 -> 0.111111111111; geometry collision sphere radius=0.0625; visual box size=0.125 0.0125 0.00625
- link spine_link_5: mass 0.1 -> 0.111111111111; geometry collision sphere radius=0.0625; visual box size=0.125 0.0125 0.00625
- link spine_link_6: mass 0.1 -> 0.111111111111; geometry collision sphere radius=0.0625; visual box size=0.125 0.0125 0.00625
- link spine_link_7: mass 0.1 -> 0.111111111111; geometry collision sphere radius=0.0625; visual box size=0.125 0.0125 0.00625
- link spine_link_8: mass 0.1 -> 0.111111111111; geometry collision sphere radius=0.0625; visual box size=0.125 0.0125 0.00625
Joints:
- joint left_girdle_abduction_joint: child left_leg -> left_girdle_connection_1; origin xyz=0 0 0 rpy=-1.570795 0 0 -> xyz=0 0.0625 0 rpy=0 0 1.570795; parent left_girdle_connection_1 -> girdle
- joint left_girdle_flection_joint: child left_girdle_connection_1 -> left_leg; limit lower=-0.523598333333 upper=1.570795 effort=30 velocity=1.0 -> lower=-1.570795 upper=1.570795 effort=30 velocity=1.0; origin xyz=0 0.125 0 rpy=0 1.570795 1.570795 -> xyz=0 0 0 rpy=1.570795 0 0; parent girdle -> left_girdle_connection_1
- joint right_girdle_abduction_joint: child right_leg -> right_girdle_connection_1; origin xyz=0 0 0 rpy=1.570795 0 0 -> xyz=0 -0.0625 0 rpy=0 0 -1.570795; parent right_girdle_connection_1 -> girdle
- joint right_girdle_flection_joint: child right_girdle_connection_1 -> right_leg; limit lower=-0.523598333333 upper=1.570795 effort=30 velocity=1.0 -> lower=-1.570795 upper=1.570795 effort=30 velocity=1.0; origin xyz=0 -0.125 0 rpy=0 1.570795 -1.570795 -> xyz=0 0 0 rpy=-1.570795 0 0; parent girdle -> right_girdle_connection_1
- joint spine_dorsal_joint_1: origin xyz=-0.125 0 0 rpy=-1.570795 0 0 -> xyz=-0.0625 0 0 rpy=-1.570795 0 0
- joint spine_dorsal_joint_2: origin xyz=-0.142857142857 0 0 rpy=-1.570795 0 0 -> xyz=-0.125 0 0 rpy=-1.570795 0 0
- joint spine_dorsal_joint_3: origin xyz=-0.142857142857 0 0 rpy=-1.570795 0 0 -> xyz=-0.125 0 0 rpy=-1.570795 0 0
- joint spine_dorsal_joint_4: origin xyz=-0.142857142857 0 0 rpy=-1.570795 0 0 -> xyz=-0.125 0 0 rpy=-1.570795 0 0
- joint spine_dorsal_joint_5: origin xyz=-0.142857142857 0 0 rpy=-1.570795 0 0 -> xyz=-0.125 0 0 rpy=-1.570795 0 0
- joint spine_dorsal_joint_6: origin xyz=-0.142857142857 0 0 rpy=-1.570795 0 0 -> xyz=-0.125 0 0 rpy=-1.570795 0 0
- joint spine_dorsal_joint_7: origin xyz=-0.142857142857 0 0 rpy=-1.570795 0 0 -> xyz=-0.125 0 0 rpy=-1.570795 0 0
- joint spine_dorsal_joint_8: origin xyz=-0.142857142857 0 0 rpy=-1.570795 0 0 -> xyz=-0.125 0 0 rpy=-1.570795 0 0

File: crawler.urdf.xacro (robot description, xacro)
@@ -8,17 +8,16 @@
   <xacro:property name="BODY_LENGTH" value="1"/>
   <xacro:property name="BODY_MASS" value="1"/>
-  <!-- NOTE: The numbers of spine segments, for now, must be matched manually to the number of macro called to add the spine segments-->
-  <xacro:property name="SPINE_SEGMENTS_NUMBER" value="7" />
+  <xacro:property name="SPINE_SEGMENTS_NUMBER" value="8" />
   <xacro:property name="SPINE_SEGMENT_LENGTH" value="${BODY_LENGTH/SPINE_SEGMENTS_NUMBER}" />
   <xacro:property name="SPINE_DORSAL_BENDING_LIMIT" value="${PI/8}" />
   <xacro:property name="SPINE_LATERAL_BENDING_LIMIT" value="${PI/4}" />
-  <xacro:property name="BODY_SPHERE_MASS" value="${BODY_MASS/(SPINE_SEGMENTS_NUMBER+3)}" /><!-- +3 for the head and girdle masses-->
+  <xacro:property name="BODY_SPHERE_MASS" value="${BODY_MASS/(SPINE_SEGMENTS_NUMBER+1)}" /><!-- +1 for the girdle masses-->
   <xacro:property name="BODY_SPHERE_RADIUS" value="${SPINE_SEGMENT_LENGTH/2}" />
   <xacro:property name="BODY_SPHERE_INERTIA" value="${2*BODY_SPHERE_MASS*BODY_SPHERE_RADIUS*BODY_SPHERE_RADIUS/5}" />
-  <xacro:property name="GIRDLE_WIDTH" value="${BODY_LENGTH/8}" />
-  <xacro:property name="GIRDLE_LENGTH" value="${BODY_LENGTH/8}" />
-  <xacro:property name="LEG_LENGTH" value="${BODY_LENGTH/10}" />
-  <xacro:property name="LEG_TIP_MASS" value="${BODY_MASS/20}" />
-  <xacro:property name="LEG_TIP_RADIUS" value="${SPINE_SEGMENT_LENGTH/4}" />
+  <xacro:property name="GIRDLE_WIDTH" value="${SPINE_SEGMENT_LENGTH/2}" />
+  <xacro:property name="GIRDLE_LENGTH" value="${SPINE_SEGMENT_LENGTH/2}" />
+  <xacro:property name="LEG_LENGTH" value="${BODY_LENGTH/8}" />
+  <xacro:property name="LEG_TIP_MASS" value="${BODY_SPHERE_MASS/10}" />
+  <xacro:property name="LEG_TIP_RADIUS" value="${BODY_SPHERE_RADIUS/3}" />
   <xacro:property name="LEG_TIP_INERTIA" value="${2*LEG_TIP_MASS*LEG_TIP_RADIUS*LEG_TIP_RADIUS/5}" />
   <xacro:property name="GIRDLE_FLEXION_LIMIT" value="${PI/2}" />
@@ -28,5 +27,5 @@
   <xacro:property name="JOINT_DAMPING" value="0.01" />
   <xacro:property name="JOINT_FRICTION" value="0.01" />
-  <xacro:property name="VISUAL_BOX_RATIO" value="0.2" />
+  <xacro:property name="VISUAL_BOX_RATIO" value="0.1" />
 <!--########### COLORS used for the links ###########-->
 <!--colors are currently implemented as macro because just defining them, as shown in the ROS tutorial, seems not to work-->
@@ -113,15 +112,16 @@
       <inertial>
         <origin xyz="0 0 0" rpy="0 0 0"/>
-        <mass value="0.01"/>
-        <inertia ixx="0.001"  ixy="0"  ixz="0" iyy="0.001" iyz="0" izz="0.001" />
-      </inertial>
-    </link>
-    <joint name="${prefix}_girdle_flection_joint" type="revolute">
-      <origin xyz="0 ${-reflect*GIRDLE_WIDTH} 0" rpy="0 ${PI/2} ${-reflect*PI/2}"/>
+        <mass value="${LEG_TIP_MASS/100}"/>
+        <inertia ixx="${LEG_TIP_INERTIA/100}"  ixy="0"  ixz="0" iyy="${LEG_TIP_INERTIA/100}" iyz="0" izz="${LEG_TIP_INERTIA/100}" />
+      </inertial>
+    </link>
+    <!--NOTE: currently leg joints have symmetrical limits, to avoid problem deriving from having symmetrical reference frame-->
+    <joint name="${prefix}_girdle_abduction_joint" type="revolute">
+      <origin xyz="0 ${-reflect*GIRDLE_WIDTH} 0" rpy="0 0 ${-reflect*PI/2}"/>
       <axis xyz="0 0 1"/>
       <parent link="girdle"/>
       <child link="${prefix}_girdle_connection_1"/>
       <dynamics damping="${JOINT_DAMPING}" friction="${JOINT_FRICTION}"/>
-      <limit effort="30" velocity="1.0" lower="-${GIRDLE_EXTENSION_LIMIT}" upper="${GIRDLE_FLEXION_LIMIT}" />
+      <limit effort="30" velocity="1.0" lower="-${GIRDLE_ABDUCTION_LIMIT}" upper="${GIRDLE_ABDUCTION_LIMIT}" />
     </joint>
     <link name="${prefix}_leg">
@@ -152,17 +152,18 @@
       </collision>
     </link>
-    <joint name="${prefix}_girdle_abduction_joint" type="revolute">
-      <origin xyz="0 0 0" rpy="${reflect*PI/2} 0 0"/>
+    <!--NOTE: currently leg joints have symmetrical limits, to avoid problem deriving from having symmetrical reference frame-->
+    <joint name="${prefix}_girdle_flection_joint" type="revolute">
+      <origin xyz="0 0 0" rpy="${-reflect*PI/2} 0 0"/>
       <axis xyz="0 0 1"/>
       <parent link="${prefix}_girdle_connection_1"/>
       <child link="${prefix}_leg"/>
       <dynamics damping="${JOINT_DAMPING}" friction="${JOINT_FRICTION}"/>
-      <limit effort="30" velocity="1.0" lower="-${GIRDLE_ADDUCTION_LIMIT}" upper="${GIRDLE_ABDUCTION_LIMIT}" />
-    </joint>
-  </xacro:macro>
-  <!-- Loop is off by one because forst segments is added manually -->
+      <limit effort="30" velocity="1.0" lower="-${GIRDLE_FLEXION_LIMIT}" upper="${GIRDLE_FLEXION_LIMIT}" />
+    </joint>
+  </xacro:macro>
+  <!-- Loop is off by one because the first segment is added manually -->
   <xacro:macro name="spine_segments_loop" params="segments_qty">
     <xacro:spine_segment_macro N="${SPINE_SEGMENTS_NUMBER + 2 - segments_qty}"/>
-    <xacro:if value="${segments_qty-1}">
+    <xacro:if value="${segments_qty-2}">
         <xacro:spine_segments_loop segments_qty="${segments_qty-1}" />
     </xacro:if>
@@ -171,31 +172,46 @@
   <link name="girdle">
    <inertial>
-     <origin xyz="0.1 0 0" rpy="0 0 0"/>
+     <origin xyz="0 0 0" rpy="0 0 0"/>
      <mass value="${BODY_SPHERE_MASS}"/>
-     <inertia ixx="${BODY_SPHERE_INERTIA}"  ixy="0"  ixz="0" iyy="${BODY_SPHERE_INERTIA}" iyz="0" izz="${BODY_SPHERE_INERTIA}" />
+     <inertia ixx="${2*BODY_SPHERE_INERTIA}"  ixy="0"  ixz="0"
+              iyy="${2*(BODY_SPHERE_INERTIA+GIRDLE_LENGTH*GIRDLE_LENGTH*BODY_SPHERE_MASS)}" iyz="0"
+              izz="${2*(BODY_SPHERE_INERTIA+GIRDLE_LENGTH*GIRDLE_LENGTH*BODY_SPHERE_MASS)}" />
    </inertial>
    <visual>
+     <origin xyz="${GIRDLE_LENGTH} 0 0" rpy="0 0 0"/>
+     <geometry>
+       <sphere radius="${BODY_SPHERE_RADIUS}" />
+     </geometry>
+     <xacro:girdle_material/>
+   </visual>
+   <visual>
+     <origin xyz="${-GIRDLE_LENGTH} 0 0" rpy="0 0 0"/>
+     <geometry>
+       <sphere radius="${BODY_SPHERE_RADIUS}" />
+     </geometry>
+     <xacro:girdle_material/>
+   </visual>
+   <visual>
      <origin xyz="0 0 0" rpy="0 0 0"/>
      <geometry>
-       <sphere radius="${BODY_SPHERE_RADIUS}" />
-     </geometry>
-     <xacro:girdle_material/>
+       <box size="${VISUAL_BOX_RATIO*2*GIRDLE_WIDTH} ${2*GIRDLE_WIDTH} ${VISUAL_BOX_RATIO*2*GIRDLE_WIDTH}"/>
+     </geometry>
+     <xacro:visual_box_material/>
    </visual>
    <visual>
      <origin xyz="0 0 0" rpy="0 0 0"/>
      <geometry>
-       <box size="${VISUAL_BOX_RATIO*2*GIRDLE_WIDTH} ${2*GIRDLE_WIDTH} ${VISUAL_BOX_RATIO*2*GIRDLE_WIDTH}"/>
+       <box size="${2*GIRDLE_LENGTH} ${VISUAL_BOX_RATIO*2*GIRDLE_LENGTH} ${VISUAL_BOX_RATIO*2*GIRDLE_WIDTH}"/>
      </geometry>
      <xacro:visual_box_material/>
    </visual>
-   <visual>
-     <origin xyz="0 0 0" rpy="0 0 0"/>
-     <geometry>
-       <box size="${2*GIRDLE_LENGTH} ${VISUAL_BOX_RATIO*2*GIRDLE_LENGTH} ${VISUAL_BOX_RATIO*2*GIRDLE_WIDTH}"/>
-     </geometry>
-     <xacro:visual_box_material/>
-   </visual>
    <collision>
-     <origin xyz="0 0 0" rpy="0 0 0"/>
+     <origin xyz="${GIRDLE_LENGTH} 0 0" rpy="0 0 0"/>
+     <geometry>
+       <sphere radius="${BODY_SPHERE_RADIUS}" />
+     </geometry>
+   </collision>
+   <collision>
+     <origin xyz="${-GIRDLE_LENGTH} 0 0" rpy="0 0 0"/>
      <geometry>
        <sphere radius="${BODY_SPHERE_RADIUS}" />
@@ -254,10 +270,4 @@
   </joint>
   <xacro:spine_segments_loop segments_qty="${SPINE_SEGMENTS_NUMBER}"/>
-<!--
-  <xacro:spine_segment_macro N="2"/>
-  <xacro:spine_segment_macro N="3"/>
-  <xacro:spine_segment_macro N="4"/>
-  <xacro:spine_segment_macro N="5"/>
-  -->
   <xacro:leg_macro prefix="right" reflect="1"/>
   <xacro:leg_macro prefix="left" reflect="-1"/>

Commit message: Started set up of leg control for walking

File: crawler.urdf (robot description, URDF)
Before this commit: robot crawler, 21 links, 20 joints
Joints:
- joint spine_lateral_joint_1: limit lower=-0.7853975 upper=0.7853975 effort=30 velocity=1.0 -> lower=-1.04719666667 upper=1.04719666667 effort=30 velocity=1.0
- joint spine_lateral_joint_2: limit lower=-0.7853975 upper=0.7853975 effort=30 velocity=1.0 -> lower=-1.04719666667 upper=1.04719666667 effort=30 velocity=1.0
- joint spine_lateral_joint_3: limit lower=-0.7853975 upper=0.7853975 effort=30 velocity=1.0 -> lower=-1.04719666667 upper=1.04719666667 effort=30 velocity=1.0
- joint spine_lateral_joint_4: limit lower=-0.7853975 upper=0.7853975 effort=30 velocity=1.0 -> lower=-1.04719666667 upper=1.04719666667 effort=30 velocity=1.0
- joint spine_lateral_joint_5: limit lower=-0.7853975 upper=0.7853975 effort=30 velocity=1.0 -> lower=-1.04719666667 upper=1.04719666667 effort=30 velocity=1.0
- joint spine_lateral_joint_6: limit lower=-0.7853975 upper=0.7853975 effort=30 velocity=1.0 -> lower=-1.04719666667 upper=1.04719666667 effort=30 velocity=1.0
- joint spine_lateral_joint_7: limit lower=-0.7853975 upper=0.7853975 effort=30 velocity=1.0 -> lower=-1.04719666667 upper=1.04719666667 effort=30 velocity=1.0
- joint spine_lateral_joint_8: limit lower=-0.7853975 upper=0.7853975 effort=30 velocity=1.0 -> lower=-1.04719666667 upper=1.04719666667 effort=30 velocity=1.0

File: crawler.urdf.xacro (robot description, xacro)
@@ -11,5 +11,5 @@
   <xacro:property name="SPINE_SEGMENT_LENGTH" value="${BODY_LENGTH/SPINE_SEGMENTS_NUMBER}" />
   <xacro:property name="SPINE_DORSAL_BENDING_LIMIT" value="${PI/8}" />
-  <xacro:property name="SPINE_LATERAL_BENDING_LIMIT" value="${PI/4}" />
+  <xacro:property name="SPINE_LATERAL_BENDING_LIMIT" value="${PI/3}" />
   <xacro:property name="BODY_SPHERE_MASS" value="${BODY_MASS/(SPINE_SEGMENTS_NUMBER+1)}" /><!-- +1 for the girdle masses-->
   <xacro:property name="BODY_SPHERE_RADIUS" value="${SPINE_SEGMENT_LENGTH/2}" />

Commit message: Single step control implemented
Discrete low pass filter for joints' speed, some preliminary study on the stability of the simulation depending on different parameters, reordered the functions of the class.
Changed the order of the spinal joints (now is lateral - dorsal)

File: crawler.urdf (robot description, URDF)
Before this commit: robot crawler, 21 links, 20 joints
Joints:
- joint spine_dorsal_joint_1: child spine_connection_1 -> spine_link_1; origin xyz=-0.0625 0 0 rpy=-1.570795 0 0 -> xyz=0 0 0 rpy=-1.570795 0 0; parent girdle -> spine_connection_1
- joint spine_dorsal_joint_2: child spine_connection_2 -> spine_link_2; origin xyz=-0.125 0 0 rpy=-1.570795 0 0 -> xyz=0 0 0 rpy=-1.570795 0 0; parent spine_link_1 -> spine_connection_2
- joint spine_dorsal_joint_3: child spine_connection_3 -> spine_link_3; origin xyz=-0.125 0 0 rpy=-1.570795 0 0 -> xyz=0 0 0 rpy=-1.570795 0 0; parent spine_link_2 -> spine_connection_3
- joint spine_dorsal_joint_4: child spine_connection_4 -> spine_link_4; origin xyz=-0.125 0 0 rpy=-1.570795 0 0 -> xyz=0 0 0 rpy=-1.570795 0 0; parent spine_link_3 -> spine_connection_4
- joint spine_dorsal_joint_5: child spine_connection_5 -> spine_link_5; origin xyz=-0.125 0 0 rpy=-1.570795 0 0 -> xyz=0 0 0 rpy=-1.570795 0 0; parent spine_link_4 -> spine_connection_5
- joint spine_dorsal_joint_6: child spine_connection_6 -> spine_link_6; origin xyz=-0.125 0 0 rpy=-1.570795 0 0 -> xyz=0 0 0 rpy=-1.570795 0 0; parent spine_link_5 -> spine_connection_6
- joint spine_dorsal_joint_7: child spine_connection_7 -> spine_link_7; origin xyz=-0.125 0 0 rpy=-1.570795 0 0 -> xyz=0 0 0 rpy=-1.570795 0 0; parent spine_link_6 -> spine_connection_7
- joint spine_dorsal_joint_8: child spine_connection_8 -> spine_link_8; origin xyz=-0.125 0 0 rpy=-1.570795 0 0 -> xyz=0 0 0 rpy=-1.570795 0 0; parent spine_link_7 -> spine_connection_8
- joint spine_lateral_joint_1: child spine_link_1 -> spine_connection_1; origin xyz=0 0 0 rpy=1.570795 0 0 -> xyz=-0.0625 0 0 rpy=0 0 0; parent spine_connection_1 -> girdle
- joint spine_lateral_joint_2: child spine_link_2 -> spine_connection_2; origin xyz=0 0 0 rpy=1.570795 0 0 -> xyz=-0.125 0 0 rpy=1.570795 0 0; parent spine_connection_2 -> spine_link_1
- joint spine_lateral_joint_3: child spine_link_3 -> spine_connection_3; origin xyz=0 0 0 rpy=1.570795 0 0 -> xyz=-0.125 0 0 rpy=1.570795 0 0; parent spine_connection_3 -> spine_link_2
- joint spine_lateral_joint_4: child spine_link_4 -> spine_connection_4; origin xyz=0 0 0 rpy=1.570795 0 0 -> xyz=-0.125 0 0 rpy=1.570795 0 0; parent spine_connection_4 -> spine_link_3
- joint spine_lateral_joint_5: child spine_link_5 -> spine_connection_5; origin xyz=0 0 0 rpy=1.570795 0 0 -> xyz=-0.125 0 0 rpy=1.570795 0 0; parent spine_connection_5 -> spine_link_4
- joint spine_lateral_joint_6: child spine_link_6 -> spine_connection_6; origin xyz=0 0 0 rpy=1.570795 0 0 -> xyz=-0.125 0 0 rpy=1.570795 0 0; parent spine_connection_6 -> spine_link_5
- joint spine_lateral_joint_7: child spine_link_7 -> spine_connection_7; origin xyz=0 0 0 rpy=1.570795 0 0 -> xyz=-0.125 0 0 rpy=1.570795 0 0; parent spine_connection_7 -> spine_link_6
- joint spine_lateral_joint_8: child spine_link_8 -> spine_connection_8; origin xyz=0 0 0 rpy=1.570795 0 0 -> xyz=-0.125 0 0 rpy=1.570795 0 0; parent spine_connection_8 -> spine_link_7

File: crawler.urdf.xacro (robot description, xacro)
@@ -91,19 +91,19 @@
       </collision>
     </link>
-    <joint name="spine_dorsal_joint_${N}" type="revolute">
-      <origin xyz="${-SPINE_SEGMENT_LENGTH} 0 0" rpy="${-PI/2} 0 0"/>
+    <joint name="spine_lateral_joint_${N}" type="revolute">
+      <origin xyz="${-SPINE_SEGMENT_LENGTH} 0 0" rpy="${PI/2} 0 0"/>
       <axis xyz="0 0 1"/>
       <parent link="spine_link_${N-1}"/>
       <child link="spine_connection_${N}"/>
       <dynamics damping="${JOINT_DAMPING}" friction="${JOINT_FRICTION}"/>
-      <limit effort="30" velocity="1.0" lower="-${SPINE_DORSAL_BENDING_LIMIT}" upper="${SPINE_DORSAL_BENDING_LIMIT}" />
-    </joint>
-    <joint name="spine_lateral_joint_${N}" type="revolute">
-      <origin xyz="0 0 0" rpy="${PI/2} 0 0"/>
+      <limit effort="30" velocity="1.0" lower="-${SPINE_LATERAL_BENDING_LIMIT}" upper="${SPINE_LATERAL_BENDING_LIMIT}" />
+    </joint>
+    <joint name="spine_dorsal_joint_${N}" type="revolute">
+      <origin xyz="0 0 0" rpy="${-PI/2} 0 0"/>
       <axis xyz="0 0 1"/>
       <parent link="spine_connection_${N}"/>
       <child link="spine_link_${N}"/>
       <dynamics damping="${JOINT_DAMPING}" friction="${JOINT_FRICTION}"/>
-      <limit effort="30" velocity="1.0" lower="-${SPINE_LATERAL_BENDING_LIMIT}" upper="${SPINE_LATERAL_BENDING_LIMIT}" />
+      <limit effort="30" velocity="1.0" lower="-${SPINE_DORSAL_BENDING_LIMIT}" upper="${SPINE_DORSAL_BENDING_LIMIT}" />
     </joint>
   </xacro:macro>
@@ -116,5 +116,5 @@
       </inertial>
     </link>
-    <!--NOTE: currently leg joints have symmetrical limits, to avoid problem deriving from having symmetrical reference frame-->
+    <!--NOTE: currently leg joints have symmetrical limits, to avoid problems deriving from having reflected reference frames-->
     <joint name="${prefix}_girdle_abduction_joint" type="revolute">
       <origin xyz="0 ${-reflect*GIRDLE_WIDTH} 0" rpy="0 0 ${-reflect*PI/2}"/>
@@ -152,5 +152,5 @@
       </collision>
     </link>
-    <!--NOTE: currently leg joints have symmetrical limits, to avoid problem deriving from having symmetrical reference frame-->
+    <!--NOTE: currently leg joints have symmetrical limits, to avoid problems deriving from having reflected reference frames-->
     <joint name="${prefix}_girdle_flection_joint" type="revolute">
       <origin xyz="0 0 0" rpy="${-reflect*PI/2} 0 0"/>
@@ -253,19 +253,19 @@
     </collision>
   </link>
-  <joint name="spine_dorsal_joint_1" type="revolute">
-    <origin xyz="${-GIRDLE_LENGTH} 0 0" rpy="${-PI/2} 0 0"/>
+  <joint name="spine_lateral_joint_1" type="revolute">
+    <origin xyz="${-GIRDLE_LENGTH} 0 0" rpy="0 0 0"/>
     <axis xyz="0 0 1"/>
     <parent link="girdle"/>
     <child link="spine_connection_1"/>
     <dynamics damping="${JOINT_DAMPING}" friction="${JOINT_FRICTION}"/>
-    <limit effort="30" velocity="1.0" lower="-${SPINE_DORSAL_BENDING_LIMIT}" upper="${SPINE_DORSAL_BENDING_LIMIT}" />
+    <limit effort="30" velocity="1.0" lower="-${SPINE_LATERAL_BENDING_LIMIT}" upper="${SPINE_LATERAL_BENDING_LIMIT}" />
   </joint>
-  <joint name="spine_lateral_joint_1" type="revolute">
-    <origin xyz="0 0 0" rpy="${PI/2} 0 0"/>
+  <joint name="spine_dorsal_joint_1" type="revolute">
+    <origin xyz="0 0 0" rpy="${-PI/2} 0 0"/>
     <axis xyz="0 0 1"/>
     <parent link="spine_connection_1"/>
     <child link="spine_link_1"/>
     <dynamics damping="${JOINT_DAMPING}" friction="${JOINT_FRICTION}"/>
-    <limit effort="30" velocity="1.0" lower="-${SPINE_LATERAL_BENDING_LIMIT}" upper="${SPINE_LATERAL_BENDING_LIMIT}" />
+    <limit effort="30" velocity="1.0" lower="-${SPINE_DORSAL_BENDING_LIMIT}" upper="${SPINE_DORSAL_BENDING_LIMIT}" />
   </joint>
   <xacro:spine_segments_loop segments_qty="${SPINE_SEGMENTS_NUMBER}"/>
