Commit message: Torque control and more

File: crawler.urdf (robot description, URDF)
Before this commit: robot crawler, 21 links, 20 joints
Links:
- link girdle: mass 0.111111111111 -> 0.1111111111111111
- link left_girdle_connection_1: mass 0.000111111111111 -> 0.0001111111111111111
- link left_leg: mass 0.0111111111111 -> 0.01111111111111111; geometry collision sphere radius=0.020833333333333332; visual box size=0.125 0.0125 0.0125
- link right_girdle_connection_1: mass 0.000111111111111 -> 0.0001111111111111111
- link right_leg: mass 0.0111111111111 -> 0.01111111111111111; geometry collision sphere radius=0.020833333333333332; visual box size=0.125 0.0125 0.0125
- link spine_connection_1: mass 0.00111111111111 -> 0.0011111111111111111
- link spine_connection_2: mass 0.00111111111111 -> 0.0011111111111111111
- link spine_connection_3: mass 0.00111111111111 -> 0.0011111111111111111
- link spine_connection_4: mass 0.00111111111111 -> 0.0011111111111111111
- link spine_connection_5: mass 0.00111111111111 -> 0.0011111111111111111
- link spine_connection_6: mass 0.00111111111111 -> 0.0011111111111111111
- link spine_connection_7: mass 0.00111111111111 -> 0.0011111111111111111
- link spine_connection_8: mass 0.00111111111111 -> 0.0011111111111111111
- link spine_link_1: mass 0.111111111111 -> 0.1111111111111111
- link spine_link_2: mass 0.111111111111 -> 0.1111111111111111
- link spine_link_3: mass 0.111111111111 -> 0.1111111111111111
- link spine_link_4: mass 0.111111111111 -> 0.1111111111111111
- link spine_link_5: mass 0.111111111111 -> 0.1111111111111111
- link spine_link_6: mass 0.111111111111 -> 0.1111111111111111
- link spine_link_7: mass 0.111111111111 -> 0.1111111111111111
- link spine_link_8: mass 0.111111111111 -> 0.1111111111111111
Joints:
- joint spine_lateral_joint_1: limit lower=-1.04719666667 upper=1.04719666667 effort=30 velocity=1.0 -> lower=-1.0471966666666666 upper=1.0471966666666666 effort=30 velocity=1.0
- joint spine_lateral_joint_2: limit lower=-1.04719666667 upper=1.04719666667 effort=30 velocity=1.0 -> lower=-1.0471966666666666 upper=1.0471966666666666 effort=30 velocity=1.0
- joint spine_lateral_joint_3: limit lower=-1.04719666667 upper=1.04719666667 effort=30 velocity=1.0 -> lower=-1.0471966666666666 upper=1.0471966666666666 effort=30 velocity=1.0
- joint spine_lateral_joint_4: limit lower=-1.04719666667 upper=1.04719666667 effort=30 velocity=1.0 -> lower=-1.0471966666666666 upper=1.0471966666666666 effort=30 velocity=1.0
- joint spine_lateral_joint_5: limit lower=-1.04719666667 upper=1.04719666667 effort=30 velocity=1.0 -> lower=-1.0471966666666666 upper=1.0471966666666666 effort=30 velocity=1.0
- joint spine_lateral_joint_6: limit lower=-1.04719666667 upper=1.04719666667 effort=30 velocity=1.0 -> lower=-1.0471966666666666 upper=1.0471966666666666 effort=30 velocity=1.0
- joint spine_lateral_joint_7: limit lower=-1.04719666667 upper=1.04719666667 effort=30 velocity=1.0 -> lower=-1.0471966666666666 upper=1.0471966666666666 effort=30 velocity=1.0
- joint spine_lateral_joint_8: limit lower=-1.04719666667 upper=1.04719666667 effort=30 velocity=1.0 -> lower=-1.0471966666666666 upper=1.0471966666666666 effort=30 velocity=1.0

Commit message: Sliding-mode torque control, PD-control, P_vel control

File: crawler.urdf (robot description, URDF)
Before this commit: robot crawler, 21 links, 20 joints
Links:
- link left_leg: geometry collision sphere radius=0.020833333333333332; visual box size=0.16666666666666666 0.016666666666666666 0.0166666666666666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
- link right_leg: geometry collision sphere radius=0.020833333333333332; visual box size=0.16666666666666666 0.016666666666666666 0.0166666666666666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
Joints:
- joint spine_lateral_joint_1: limit lower=-1.0471966666666666 upper=1.0471966666666666 effort=30 velocity=1.0 -> lower=-1.570795 upper=1.570795 effort=30 velocity=1.0
- joint spine_lateral_joint_2: limit lower=-1.0471966666666666 upper=1.0471966666666666 effort=30 velocity=1.0 -> lower=-1.570795 upper=1.570795 effort=30 velocity=1.0
- joint spine_lateral_joint_3: limit lower=-1.0471966666666666 upper=1.0471966666666666 effort=30 velocity=1.0 -> lower=-1.570795 upper=1.570795 effort=30 velocity=1.0
- joint spine_lateral_joint_4: limit lower=-1.0471966666666666 upper=1.0471966666666666 effort=30 velocity=1.0 -> lower=-1.570795 upper=1.570795 effort=30 velocity=1.0
- joint spine_lateral_joint_5: limit lower=-1.0471966666666666 upper=1.0471966666666666 effort=30 velocity=1.0 -> lower=-1.570795 upper=1.570795 effort=30 velocity=1.0
- joint spine_lateral_joint_6: limit lower=-1.0471966666666666 upper=1.0471966666666666 effort=30 velocity=1.0 -> lower=-1.570795 upper=1.570795 effort=30 velocity=1.0
- joint spine_lateral_joint_7: limit lower=-1.0471966666666666 upper=1.0471966666666666 effort=30 velocity=1.0 -> lower=-1.570795 upper=1.570795 effort=30 velocity=1.0
- joint spine_lateral_joint_8: limit lower=-1.0471966666666666 upper=1.0471966666666666 effort=30 velocity=1.0 -> lower=-1.570795 upper=1.570795 effort=30 velocity=1.0

File: crawler.urdf.xacro (robot description, xacro)
@@ -11,5 +11,5 @@
   <xacro:property name="SPINE_SEGMENT_LENGTH" value="${BODY_LENGTH/SPINE_SEGMENTS_NUMBER}" />
   <xacro:property name="SPINE_DORSAL_BENDING_LIMIT" value="${PI/8}" />
-  <xacro:property name="SPINE_LATERAL_BENDING_LIMIT" value="${PI/3}" />
+  <xacro:property name="SPINE_LATERAL_BENDING_LIMIT" value="${PI/2}" />
   <xacro:property name="BODY_SPHERE_MASS" value="${BODY_MASS/(SPINE_SEGMENTS_NUMBER+1)}" /><!-- +1 for the girdle masses-->
   <xacro:property name="BODY_SPHERE_RADIUS" value="${SPINE_SEGMENT_LENGTH/2}" />
@@ -17,5 +17,5 @@
   <xacro:property name="GIRDLE_WIDTH" value="${SPINE_SEGMENT_LENGTH/2}" />
   <xacro:property name="GIRDLE_LENGTH" value="${SPINE_SEGMENT_LENGTH/2}" />
-  <xacro:property name="LEG_LENGTH" value="${BODY_LENGTH/8}" />
+  <xacro:property name="LEG_LENGTH" value="${BODY_LENGTH/6}" />
   <xacro:property name="LEG_TIP_MASS" value="${BODY_SPHERE_MASS/10}" />
   <xacro:property name="LEG_TIP_RADIUS" value="${BODY_SPHERE_RADIUS/3}" />

Commit message: Code for animations, various trial of control with different URDF

File: crawler.urdf (robot description, URDF)
Before this commit: robot crawler, 21 links, 20 joints
Links:
- removed link spine_connection_3
- removed link spine_connection_4
- removed link spine_connection_5
- removed link spine_connection_6
- removed link spine_connection_7
- removed link spine_connection_8
- removed link spine_link_3
- removed link spine_link_4
- removed link spine_link_5
- removed link spine_link_6
- removed link spine_link_7
- removed link spine_link_8
- link girdle: mass 0.1111111111111111 -> 0.3333333333333333; geometry collision sphere radius=0.0625; collision sphere radius=0.0625
- link left_girdle_connection_1: mass 0.0001111111111111111 -> 0.0003333333333333333
- link left_leg: mass 0.01111111111111111 -> 0.03333333333333333
- link right_girdle_connection_1: mass 0.0001111111111111111 -> 0.0003333333333333333
- link right_leg: mass 0.01111111111111111 -> 0.03333333333333333
- link spine_connection_1: mass 0.0011111111111111111 -> 0.003333333333333333
- link spine_connection_2: mass 0.0011111111111111111 -> 0.003333333333333333
- link spine_link_1: mass 0.1111111111111111 -> 0.3333333333333333; geometry collision sphere radius=0.0625; visual box size=0.5 0.05 0.00625
- link spine_link_2: mass 0.1111111111111111 -> 0.3333333333333333; geometry collision sphere radius=0.0625; visual box size=0.5 0.05 0.00625
Joints:
- removed joint spine_dorsal_joint_3
- removed joint spine_dorsal_joint_4
- removed joint spine_dorsal_joint_5
- removed joint spine_dorsal_joint_6
- removed joint spine_dorsal_joint_7
- removed joint spine_dorsal_joint_8
- removed joint spine_lateral_joint_3
- removed joint spine_lateral_joint_4
- removed joint spine_lateral_joint_5
- removed joint spine_lateral_joint_6
- removed joint spine_lateral_joint_7
- removed joint spine_lateral_joint_8
- joint spine_lateral_joint_1: origin xyz=-0.0625 0 0 rpy=0 0 0 -> xyz=-0.25 0 0 rpy=0 0 0
- joint spine_lateral_joint_2: origin xyz=-0.125 0 0 rpy=1.570795 0 0 -> xyz=-0.5 0 0 rpy=1.570795 0 0

File: crawler.urdf.xacro (robot description, xacro)
@@ -8,12 +8,12 @@
   <xacro:property name="BODY_LENGTH" value="1"/>
   <xacro:property name="BODY_MASS" value="1"/>
-  <xacro:property name="SPINE_SEGMENTS_NUMBER" value="8" />
+  <xacro:property name="SPINE_SEGMENTS_NUMBER" value="2" />
   <xacro:property name="SPINE_SEGMENT_LENGTH" value="${BODY_LENGTH/SPINE_SEGMENTS_NUMBER}" />
   <xacro:property name="SPINE_DORSAL_BENDING_LIMIT" value="${PI/8}" />
   <xacro:property name="SPINE_LATERAL_BENDING_LIMIT" value="${PI/2}" />
   <xacro:property name="BODY_SPHERE_MASS" value="${BODY_MASS/(SPINE_SEGMENTS_NUMBER+1)}" /><!-- +1 for the girdle masses-->
-  <xacro:property name="BODY_SPHERE_RADIUS" value="${SPINE_SEGMENT_LENGTH/2}" />
+  <xacro:property name="BODY_SPHERE_RADIUS" value="${BODY_LENGTH/16}" />
   <xacro:property name="BODY_SPHERE_INERTIA" value="${2*BODY_SPHERE_MASS*BODY_SPHERE_RADIUS*BODY_SPHERE_RADIUS/5}" />
-  <xacro:property name="GIRDLE_WIDTH" value="${SPINE_SEGMENT_LENGTH/2}" />
+  <xacro:property name="GIRDLE_WIDTH" value="${BODY_LENGTH/16}" />
   <xacro:property name="GIRDLE_LENGTH" value="${SPINE_SEGMENT_LENGTH/2}" />
   <xacro:property name="LEG_LENGTH" value="${BODY_LENGTH/6}" />

Commit message: Videos of simulation, animations and other stuff

File: crawler.urdf (robot description, URDF)
Before this commit: robot crawler, 9 links, 8 joints
Links:
- added link spine_connection_3, mass 0.00125
- added link spine_connection_4, mass 0.00125
- added link spine_connection_5, mass 0.00125
- added link spine_connection_6, mass 0.00125
- added link spine_connection_7, mass 0.00125
- added link spine_link_3, mass 0.125; collision sphere radius=0.03125; visual box size=0.0714285714286 0.00357142857143 0.00357142857143
- added link spine_link_4, mass 0.125; collision sphere radius=0.03125; visual box size=0.0714285714286 0.00357142857143 0.00357142857143
- added link spine_link_5, mass 0.125; collision sphere radius=0.03125; visual box size=0.0714285714286 0.00357142857143 0.00357142857143
- added link spine_link_6, mass 0.125; collision sphere radius=0.03125; visual box size=0.0714285714286 0.00357142857143 0.00357142857143
- added link spine_link_7, mass 0.125; collision sphere radius=0.03125; visual box size=0.0714285714286 0.00357142857143 0.00357142857143
- link girdle: mass 0.3333333333333333 -> 0.125; geometry collision sphere radius=0.03125; collision sphere radius=0.03125
- link left_girdle_connection_1: mass 0.0003333333333333333 -> 0.000125
- link left_leg: mass 0.03333333333333333 -> 0.0125; geometry collision sphere radius=0.0104166666667; visual box size=0.0625 0.003125 0.003125
- link right_girdle_connection_1: mass 0.0003333333333333333 -> 0.000125
- link right_leg: mass 0.03333333333333333 -> 0.0125; geometry collision sphere radius=0.0104166666667; visual box size=0.0625 0.003125 0.003125
- link spine_connection_1: mass 0.003333333333333333 -> 0.00125
- link spine_connection_2: mass 0.003333333333333333 -> 0.00125
- link spine_link_1: mass 0.3333333333333333 -> 0.125; geometry collision sphere radius=0.03125; visual box size=0.0714285714286 0.00357142857143 0.00357142857143
- link spine_link_2: mass 0.3333333333333333 -> 0.125; geometry collision sphere radius=0.03125; visual box size=0.0714285714286 0.00357142857143 0.00357142857143
Joints:
- added joint spine_dorsal_joint_3: type revolute, parent spine_connection_3, child spine_link_3, origin xyz=0 0 0 rpy=-1.570795 0 0, axis 0 0 1, limit lower=-0.39269875 upper=0.39269875 effort=30 velocity=1.0
- added joint spine_dorsal_joint_4: type revolute, parent spine_connection_4, child spine_link_4, origin xyz=0 0 0 rpy=-1.570795 0 0, axis 0 0 1, limit lower=-0.39269875 upper=0.39269875 effort=30 velocity=1.0
- added joint spine_dorsal_joint_5: type revolute, parent spine_connection_5, child spine_link_5, origin xyz=0 0 0 rpy=-1.570795 0 0, axis 0 0 1, limit lower=-0.39269875 upper=0.39269875 effort=30 velocity=1.0
- added joint spine_dorsal_joint_6: type revolute, parent spine_connection_6, child spine_link_6, origin xyz=0 0 0 rpy=-1.570795 0 0, axis 0 0 1, limit lower=-0.39269875 upper=0.39269875 effort=30 velocity=1.0
- added joint spine_dorsal_joint_7: type revolute, parent spine_connection_7, child spine_link_7, origin xyz=0 0 0 rpy=-1.570795 0 0, axis 0 0 1, limit lower=-0.39269875 upper=0.39269875 effort=30 velocity=1.0
- added joint spine_lateral_joint_3: type revolute, parent spine_link_2, child spine_connection_3, origin xyz=-0.0714285714286 0 0 rpy=1.570795 0 0, axis 0 0 1, limit lower=-1.570795 upper=1.570795 effort=30 velocity=1.0
- added joint spine_lateral_joint_4: type revolute, parent spine_link_3, child spine_connection_4, origin xyz=-0.0714285714286 0 0 rpy=1.570795 0 0, axis 0 0 1, limit lower=-1.570795 upper=1.570795 effort=30 velocity=1.0
- added joint spine_lateral_joint_5: type revolute, parent spine_link_4, child spine_connection_5, origin xyz=-0.0714285714286 0 0 rpy=1.570795 0 0, axis 0 0 1, limit lower=-1.570795 upper=1.570795 effort=30 velocity=1.0
- added joint spine_lateral_joint_6: type revolute, parent spine_link_5, child spine_connection_6, origin xyz=-0.0714285714286 0 0 rpy=1.570795 0 0, axis 0 0 1, limit lower=-1.570795 upper=1.570795 effort=30 velocity=1.0
- added joint spine_lateral_joint_7: type revolute, parent spine_link_6, child spine_connection_7, origin xyz=-0.0714285714286 0 0 rpy=1.570795 0 0, axis 0 0 1, limit lower=-1.570795 upper=1.570795 effort=30 velocity=1.0
- joint left_girdle_abduction_joint: origin xyz=0 0.0625 0 rpy=0 0 1.570795 -> xyz=0 0.03125 0 rpy=0 0 1.570795
- joint right_girdle_abduction_joint: origin xyz=0 -0.0625 0 rpy=0 0 -1.570795 -> xyz=0 -0.03125 0 rpy=0 0 -1.570795
- joint spine_lateral_joint_1: origin xyz=-0.25 0 0 rpy=0 0 0 -> xyz=-0.05 0 0 rpy=0 0 0
- joint spine_lateral_joint_2: origin xyz=-0.5 0 0 rpy=1.570795 0 0 -> xyz=-0.0714285714286 0 0 rpy=1.570795 0 0

File: crawler.urdf.xacro (robot description, xacro)
@@ -6,8 +6,8 @@
   <!--CONSTANTS-->
   <xacro:property name="PI" value="3.14159" />
-  <xacro:property name="BODY_LENGTH" value="1"/>
+  <xacro:property name="BODY_LENGTH" value="0.5"/>
   <xacro:property name="BODY_MASS" value="1"/>
-  <xacro:property name="SPINE_SEGMENTS_NUMBER" value="2" />
-  <xacro:property name="SPINE_SEGMENT_LENGTH" value="${BODY_LENGTH/SPINE_SEGMENTS_NUMBER}" />
+  <xacro:property name="SPINE_SEGMENTS_NUMBER" value="7" />
+  <xacro:property name="SPINE_SEGMENT_LENGTH" value="${BODY_LENGTH/(SPINE_SEGMENTS_NUMBER)}" />
   <xacro:property name="SPINE_DORSAL_BENDING_LIMIT" value="${PI/8}" />
   <xacro:property name="SPINE_LATERAL_BENDING_LIMIT" value="${PI/2}" />
@@ -16,6 +16,6 @@
   <xacro:property name="BODY_SPHERE_INERTIA" value="${2*BODY_SPHERE_MASS*BODY_SPHERE_RADIUS*BODY_SPHERE_RADIUS/5}" />
   <xacro:property name="GIRDLE_WIDTH" value="${BODY_LENGTH/16}" />
-  <xacro:property name="GIRDLE_LENGTH" value="${SPINE_SEGMENT_LENGTH/2}" />
-  <xacro:property name="LEG_LENGTH" value="${BODY_LENGTH/6}" />
+  <xacro:property name="GIRDLE_LENGTH" value="${BODY_LENGTH/10}" />
+  <xacro:property name="LEG_LENGTH" value="${BODY_LENGTH/8}" />
   <xacro:property name="LEG_TIP_MASS" value="${BODY_SPHERE_MASS/10}" />
   <xacro:property name="LEG_TIP_RADIUS" value="${BODY_SPHERE_RADIUS/3}" />
@@ -25,7 +25,7 @@
   <xacro:property name="GIRDLE_ABDUCTION_LIMIT" value="${PI/2}" />
   <xacro:property name="GIRDLE_ADDUCTION_LIMIT" value="${PI/2}" />
-  <xacro:property name="JOINT_DAMPING" value="0.01" />
-  <xacro:property name="JOINT_FRICTION" value="0.01" />
-  <xacro:property name="VISUAL_BOX_RATIO" value="0.1" />
+  <xacro:property name="JOINT_DAMPING" value="0.001" />
+  <xacro:property name="JOINT_FRICTION" value="0.001" />
+  <xacro:property name="VISUAL_BOX_RATIO" value="0.05" />
 <!--########### COLORS used for the links ###########-->
 <!--colors are currently implemented as macro because just defining them, as shown in the ROS tutorial, seems not to work-->
@@ -64,5 +64,5 @@
         <origin xyz="${-SPINE_SEGMENT_LENGTH/2} 0 0" rpy="0 0 0"/>
         <geometry>
-          <box size="${SPINE_SEGMENT_LENGTH} ${VISUAL_BOX_RATIO*SPINE_SEGMENT_LENGTH} ${VISUAL_BOX_RATIO*GIRDLE_WIDTH}"/>
+          <box size="${SPINE_SEGMENT_LENGTH} ${VISUAL_BOX_RATIO*SPINE_SEGMENT_LENGTH} ${VISUAL_BOX_RATIO*SPINE_SEGMENT_LENGTH}"/>
         </geometry>
       </visual>
@@ -182,5 +182,5 @@
      <origin xyz="0 0 0" rpy="0 0 0"/>
      <geometry>
-       <box size="${2*GIRDLE_LENGTH} ${VISUAL_BOX_RATIO*2*GIRDLE_LENGTH} ${VISUAL_BOX_RATIO*2*GIRDLE_WIDTH}"/>
+       <box size="${2*GIRDLE_LENGTH} ${VISUAL_BOX_RATIO*2*GIRDLE_LENGTH} ${VISUAL_BOX_RATIO*2*GIRDLE_LENGTH}"/>
      </geometry>
    </visual>
@@ -221,5 +221,5 @@
       <origin xyz="${-SPINE_SEGMENT_LENGTH/2} 0 0" rpy="0 0 0"/>
       <geometry>
-        <box size="${SPINE_SEGMENT_LENGTH} ${VISUAL_BOX_RATIO*SPINE_SEGMENT_LENGTH} ${VISUAL_BOX_RATIO*GIRDLE_WIDTH}"/>
+        <box size="${SPINE_SEGMENT_LENGTH} ${VISUAL_BOX_RATIO*SPINE_SEGMENT_LENGTH} ${VISUAL_BOX_RATIO*SPINE_SEGMENT_LENGTH}"/>
       </geometry>
     </visual>

Commit message: Framework for Bayesian Optimization added and tested

File: crawler.urdf (robot description, URDF)
Before this commit: robot crawler, 19 links, 18 joints
Links:
- removed link spine_connection_6
- removed link spine_connection_7
- removed link spine_link_6
- removed link spine_link_7
- link girdle: mass 0.125 -> 0.166666666667; geometry collision sphere radius=0.01875; collision sphere radius=0.01875
- link left_girdle_connection_1: mass 0.000125 -> 0.000166666666667
- link left_leg: mass 0.0125 -> 0.0166666666667; geometry collision sphere radius=0.00625; visual box size=0.0375 0.001875 0.001875
- link right_girdle_connection_1: mass 0.000125 -> 0.000166666666667
- link right_leg: mass 0.0125 -> 0.0166666666667; geometry collision sphere radius=0.00625; visual box size=0.0375 0.001875 0.001875
- link spine_connection_1: mass 0.00125 -> 0.00166666666667
- link spine_connection_2: mass 0.00125 -> 0.00166666666667
- link spine_connection_3: mass 0.00125 -> 0.00166666666667
- link spine_connection_4: mass 0.00125 -> 0.00166666666667
- link spine_connection_5: mass 0.00125 -> 0.00166666666667
- link spine_link_1: mass 0.125 -> 0.166666666667; geometry collision sphere radius=0.01875; visual box size=0.06 0.003 0.003
- link spine_link_2: mass 0.125 -> 0.166666666667; geometry collision sphere radius=0.01875; visual box size=0.06 0.003 0.003
- link spine_link_3: mass 0.125 -> 0.166666666667; geometry collision sphere radius=0.01875; visual box size=0.06 0.003 0.003
- link spine_link_4: mass 0.125 -> 0.166666666667; geometry collision sphere radius=0.01875; visual box size=0.06 0.003 0.003
- link spine_link_5: mass 0.125 -> 0.166666666667; geometry collision sphere radius=0.01875; visual box size=0.06 0.003 0.003
Joints:
- removed joint spine_dorsal_joint_6
- removed joint spine_dorsal_joint_7
- removed joint spine_lateral_joint_6
- removed joint spine_lateral_joint_7
- joint left_girdle_abduction_joint: origin xyz=0 0.03125 0 rpy=0 0 1.570795 -> xyz=0 0.01875 0 rpy=0 0 1.570795
- joint left_girdle_flection_joint: limit lower=-1.570795 upper=1.570795 effort=30 velocity=1.0 -> lower=-0.523598333333 upper=0.523598333333 effort=30 velocity=1.0
- joint right_girdle_abduction_joint: origin xyz=0 -0.03125 0 rpy=0 0 -1.570795 -> xyz=0 -0.01875 0 rpy=0 0 -1.570795
- joint right_girdle_flection_joint: limit lower=-1.570795 upper=1.570795 effort=30 velocity=1.0 -> lower=-0.523598333333 upper=0.523598333333 effort=30 velocity=1.0
- joint spine_lateral_joint_1: origin xyz=-0.05 0 0 rpy=0 0 0 -> xyz=-0.03 0 0 rpy=0 0 0
- joint spine_lateral_joint_2: origin xyz=-0.0714285714286 0 0 rpy=1.570795 0 0 -> xyz=-0.06 0 0 rpy=1.570795 0 0
- joint spine_lateral_joint_3: origin xyz=-0.0714285714286 0 0 rpy=1.570795 0 0 -> xyz=-0.06 0 0 rpy=1.570795 0 0
- joint spine_lateral_joint_4: origin xyz=-0.0714285714286 0 0 rpy=1.570795 0 0 -> xyz=-0.06 0 0 rpy=1.570795 0 0
- joint spine_lateral_joint_5: origin xyz=-0.0714285714286 0 0 rpy=1.570795 0 0 -> xyz=-0.06 0 0 rpy=1.570795 0 0

File: crawler.urdf.xacro (robot description, xacro)
@@ -6,7 +6,7 @@
   <!--CONSTANTS-->
   <xacro:property name="PI" value="3.14159" />
-  <xacro:property name="BODY_LENGTH" value="0.5"/>
+  <xacro:property name="BODY_LENGTH" value="0.3"/>
   <xacro:property name="BODY_MASS" value="1"/>
-  <xacro:property name="SPINE_SEGMENTS_NUMBER" value="7" />
+  <xacro:property name="SPINE_SEGMENTS_NUMBER" value="5" />
   <xacro:property name="SPINE_SEGMENT_LENGTH" value="${BODY_LENGTH/(SPINE_SEGMENTS_NUMBER)}" />
   <xacro:property name="SPINE_DORSAL_BENDING_LIMIT" value="${PI/8}" />
@@ -21,5 +21,5 @@
   <xacro:property name="LEG_TIP_RADIUS" value="${BODY_SPHERE_RADIUS/3}" />
   <xacro:property name="LEG_TIP_INERTIA" value="${2*LEG_TIP_MASS*LEG_TIP_RADIUS*LEG_TIP_RADIUS/5}" />
-  <xacro:property name="GIRDLE_FLEXION_LIMIT" value="${PI/2}" />
+  <xacro:property name="GIRDLE_FLEXION_LIMIT" value="${PI/6}" />
   <xacro:property name="GIRDLE_EXTENSION_LIMIT" value="${PI/6}" />
   <xacro:property name="GIRDLE_ABDUCTION_LIMIT" value="${PI/2}" />
