Commit message: Sim_crawler.py functions for joint control and COM tracking

File: crawler.urdf.xacro (robot description, xacro)
@@ -171,5 +171,5 @@
   <link name="girdle">
    <inertial>
-     <origin xyz="0 0 0" rpy="0 0 0"/>
+     <origin xyz="0.1 0 0" rpy="0 0 0"/>
      <mass value="${BODY_SPHERE_MASS}"/>
      <inertia ixx="${BODY_SPHERE_INERTIA}"  ixy="0"  ixz="0" iyy="${BODY_SPHERE_INERTIA}" iyz="0" izz="${BODY_SPHERE_INERTIA}" />

Commit message: Set URDF colors

File: crawler.urdf.xacro (robot description, xacro)
@@ -30,29 +30,13 @@
 <!--########### COLORS used for the links ###########-->
 <!--colors are currently implemented as macro because just defining them, as shown in the ROS tutorial, seems not to work-->
-  <xacro:macro name="girdle_material">
-    <material name="girdle_material">
-      <color rgba="0.878 0.471 0.333 0.1"/>
-    </material>
-  </xacro:macro>
-  <!--<xacro:macro name="girdle_material">
-    <material name="red">
-      <color rgba="1 0 0 0.5"/>
-    </material>
-  </xacro:macro>-->
-  <xacro:macro name="body_material">
-    <material name="body_material">
-      <color rgba="0.176 0.188 0.278 1.0"/>
-    </material>
-  </xacro:macro>
-  <xacro:macro name="leg_material">
-    <material name="leg_material">
-      <color rgba="0.106 0.6 0.545 1.0"/>
-    </material>
-  </xacro:macro>
-  <xacro:macro name="visual_box_material">
-    <material name="visual_box_material">
-      <color rgba="0.627 0.620 0.733 1.0"/>
-    </material>
-  </xacro:macro>
+  <material name="girdle_material">
+    <color rgba="0.106 0.6 0.545 1"/>
+  </material>
+  <material name="body_material">
+    <color rgba="1 0.8235 0.298 1"/>
+  </material>
+  <material name="leg_material">
+    <color rgba="0.878 0.471 0.333 1"/>
+  </material>
 <!--########### MACRO for links and joints ###########-->
   <xacro:macro name="spine_segment_macro" params="N">
@@ -75,5 +59,5 @@
           <sphere radius="${BODY_SPHERE_RADIUS}" />
         </geometry>
-        <xacro:body_material/>
+        <material name="body_material"/>
       </visual>
       <visual>
@@ -82,5 +66,4 @@
           <box size="${SPINE_SEGMENT_LENGTH} ${VISUAL_BOX_RATIO*SPINE_SEGMENT_LENGTH} ${VISUAL_BOX_RATIO*GIRDLE_WIDTH}"/>
         </geometry>
-        <xacro:visual_box_material/>
       </visual>
       <collision>
@@ -136,5 +119,5 @@
           <sphere radius="${LEG_TIP_RADIUS}" />
         </geometry>
-        <xacro:leg_material/>
+        <material name="leg_material"/>
       </visual>
       <visual>
@@ -143,5 +126,4 @@
           <box size="${LEG_LENGTH} ${VISUAL_BOX_RATIO*LEG_LENGTH} ${VISUAL_BOX_RATIO*LEG_LENGTH}" />
         </geometry>
-        <xacro:visual_box_material/>
       </visual>
       <collision>
@@ -183,5 +165,5 @@
        <sphere radius="${BODY_SPHERE_RADIUS}" />
      </geometry>
-     <xacro:girdle_material/>
+     <material name="girdle_material"/>
    </visual>
    <visual>
@@ -190,5 +172,4 @@
        <sphere radius="${BODY_SPHERE_RADIUS}" />
      </geometry>
-     <xacro:girdle_material/>
    </visual>
    <visual>
@@ -197,5 +178,4 @@
        <box size="${VISUAL_BOX_RATIO*2*GIRDLE_WIDTH} ${2*GIRDLE_WIDTH} ${VISUAL_BOX_RATIO*2*GIRDLE_WIDTH}"/>
      </geometry>
-     <xacro:visual_box_material/>
    </visual>
    <visual>
@@ -204,5 +184,4 @@
        <box size="${2*GIRDLE_LENGTH} ${VISUAL_BOX_RATIO*2*GIRDLE_LENGTH} ${VISUAL_BOX_RATIO*2*GIRDLE_WIDTH}"/>
      </geometry>
-     <xacro:visual_box_material/>
    </visual>
    <collision>
@@ -237,5 +216,5 @@
         <sphere radius="${BODY_SPHERE_RADIUS}" />
       </geometry>
-      <xacro:body_material/>
+      <material name="body_material"/>
     </visual>
     <visual>
@@ -244,5 +223,4 @@
         <box size="${SPINE_SEGMENT_LENGTH} ${VISUAL_BOX_RATIO*SPINE_SEGMENT_LENGTH} ${VISUAL_BOX_RATIO*GIRDLE_WIDTH}"/>
       </geometry>
-      <xacro:visual_box_material/>
     </visual>
     <collision>

Commit message: Multi-step simulation implemented

File: crawler.urdf.xacro (robot description, xacro)
@@ -6,7 +6,7 @@
   <!--CONSTANTS-->
   <xacro:property name="PI" value="3.14159" />
-  <xacro:property name="BODY_LENGTH" value="1"/>
+  <xacro:property name="BODY_LENGTH" value="0.5"/>
   <xacro:property name="BODY_MASS" value="1"/>
-  <xacro:property name="SPINE_SEGMENTS_NUMBER" value="8" />
+  <xacro:property name="SPINE_SEGMENTS_NUMBER" value="4" />
   <xacro:property name="SPINE_SEGMENT_LENGTH" value="${BODY_LENGTH/SPINE_SEGMENTS_NUMBER}" />
   <xacro:property name="SPINE_DORSAL_BENDING_LIMIT" value="${PI/8}" />

Commit message: Videos and test + jamming behaviour

File: crawler.urdf.xacro (robot description, xacro)
@@ -6,7 +6,7 @@
   <!--CONSTANTS-->
   <xacro:property name="PI" value="3.14159" />
-  <xacro:property name="BODY_LENGTH" value="0.5"/>
+  <xacro:property name="BODY_LENGTH" value="1"/>
   <xacro:property name="BODY_MASS" value="1"/>
-  <xacro:property name="SPINE_SEGMENTS_NUMBER" value="4" />
+  <xacro:property name="SPINE_SEGMENTS_NUMBER" value="8" />
   <xacro:property name="SPINE_SEGMENT_LENGTH" value="${BODY_LENGTH/SPINE_SEGMENTS_NUMBER}" />
   <xacro:property name="SPINE_DORSAL_BENDING_LIMIT" value="${PI/8}" />

Commit message: Traveling wave control, lot of videos, trials with big and small models

File: crawler.urdf.xacro (robot description, xacro)
@@ -6,16 +6,17 @@
   <!--CONSTANTS-->
   <xacro:property name="PI" value="3.14159" />
-  <xacro:property name="BODY_LENGTH" value="0.3"/>
-  <xacro:property name="BODY_MASS" value="1"/>
+  <xacro:property name="BODY_LENGTH" value="0.076"/>
+  <xacro:property name="BODY_MASS" value="0.0028"/>
   <xacro:property name="SPINE_SEGMENTS_NUMBER" value="5" />
-  <xacro:property name="SPINE_SEGMENT_LENGTH" value="${BODY_LENGTH/(SPINE_SEGMENTS_NUMBER)}" />
+  <xacro:property name="N_HALF" value="3" />
+  <xacro:property name="SPINE_SEGMENT_LENGTH" value="${BODY_LENGTH/(SPINE_SEGMENTS_NUMBER+1)}" />
   <xacro:property name="SPINE_DORSAL_BENDING_LIMIT" value="${PI/8}" />
   <xacro:property name="SPINE_LATERAL_BENDING_LIMIT" value="${PI/2}" />
-  <xacro:property name="BODY_SPHERE_MASS" value="${BODY_MASS/(SPINE_SEGMENTS_NUMBER+1)}" /><!-- +1 for the girdle masses-->
+  <xacro:property name="BODY_SPHERE_MASS" value="${BODY_MASS/(SPINE_SEGMENTS_NUMBER+2)}" /><!-- +2 for the girdle masses-->
   <xacro:property name="BODY_SPHERE_RADIUS" value="${BODY_LENGTH/16}" />
   <xacro:property name="BODY_SPHERE_INERTIA" value="${2*BODY_SPHERE_MASS*BODY_SPHERE_RADIUS*BODY_SPHERE_RADIUS/5}" />
-  <xacro:property name="GIRDLE_WIDTH" value="${BODY_LENGTH/16}" />
-  <xacro:property name="GIRDLE_LENGTH" value="${BODY_LENGTH/10}" />
-  <xacro:property name="LEG_LENGTH" value="${BODY_LENGTH/8}" />
+  <xacro:property name="GIRDLE_WIDTH" value="${BODY_LENGTH/14}" />
+  <xacro:property name="GIRDLE_LENGTH" value="${SPINE_SEGMENT_LENGTH/2}" />
+  <xacro:property name="LEG_LENGTH" value="${BODY_LENGTH/9.4}" />
   <xacro:property name="LEG_TIP_MASS" value="${BODY_SPHERE_MASS/10}" />
   <xacro:property name="LEG_TIP_RADIUS" value="${BODY_SPHERE_RADIUS/3}" />
@@ -25,7 +26,14 @@
   <xacro:property name="GIRDLE_ABDUCTION_LIMIT" value="${PI/2}" />
   <xacro:property name="GIRDLE_ADDUCTION_LIMIT" value="${PI/2}" />
-  <xacro:property name="JOINT_DAMPING" value="0.001" />
-  <xacro:property name="JOINT_FRICTION" value="0.001" />
+  <xacro:property name="JOINT_DAMPING" value="0.0" />
+  <xacro:property name="JOINT_FRICTION" value="0.0" />
+  <xacro:property name="JOINT_MAX_SPEED" value="50.0" />
+  <xacro:property name="JOINT_MAX_EFFORT" value="50.0" />
   <xacro:property name="VISUAL_BOX_RATIO" value="0.05" />
+  <!--MASS SCALING-->
+  <!--Values taken from the 5-bars model-->
+  <xacro:property name="KB" value="${(0.456-0.196)/(BODY_LENGTH*0.37)}" />
+  <xacro:property name="KT" value="${(0.218-0.456)/(BODY_LENGTH*0.49)}" />
+  <xacro:property name="M0" value="${(BODY_MASS - KB*SPINE_SEGMENT_LENGTH*(N_HALF*(N_HALF+1))/2 - KT*SPINE_SEGMENT_LENGTH*((SPINE_SEGMENTS_NUMBER-N_HALF)*(SPINE_SEGMENTS_NUMBER-N_HALF+1))/2)/SPINE_SEGMENTS_NUMBER}" />
 <!--########### COLORS used for the links ###########-->
 <!--colors are currently implemented as macro because just defining them, as shown in the ROS tutorial, seems not to work-->
@@ -80,5 +88,5 @@
       <child link="spine_connection_${N}"/>
       <dynamics damping="${JOINT_DAMPING}" friction="${JOINT_FRICTION}"/>
-      <limit effort="30" velocity="1.0" lower="-${SPINE_LATERAL_BENDING_LIMIT}" upper="${SPINE_LATERAL_BENDING_LIMIT}" />
+      <limit effort="${JOINT_MAX_EFFORT}" velocity="${JOINT_MAX_SPEED}" lower="-${SPINE_LATERAL_BENDING_LIMIT}" upper="${SPINE_LATERAL_BENDING_LIMIT}" />
     </joint>
     <joint name="spine_dorsal_joint_${N}" type="revolute">
@@ -88,5 +96,5 @@
       <child link="spine_link_${N}"/>
       <dynamics damping="${JOINT_DAMPING}" friction="${JOINT_FRICTION}"/>
-      <limit effort="30" velocity="1.0" lower="-${SPINE_DORSAL_BENDING_LIMIT}" upper="${SPINE_DORSAL_BENDING_LIMIT}" />
+      <limit effort="${JOINT_MAX_EFFORT}" velocity="${JOINT_MAX_SPEED}" lower="-${SPINE_DORSAL_BENDING_LIMIT}" upper="${SPINE_DORSAL_BENDING_LIMIT}" />
     </joint>
   </xacro:macro>
@@ -106,5 +114,5 @@
       <child link="${prefix}_girdle_connection_1"/>
       <dynamics damping="${JOINT_DAMPING}" friction="${JOINT_FRICTION}"/>
-      <limit effort="30" velocity="1.0" lower="-${GIRDLE_ABDUCTION_LIMIT}" upper="${GIRDLE_ABDUCTION_LIMIT}" />
+      <limit effort="${JOINT_MAX_EFFORT}" velocity="${JOINT_MAX_SPEED}" lower="-${GIRDLE_ABDUCTION_LIMIT}" upper="${GIRDLE_ABDUCTION_LIMIT}" />
     </joint>
     <link name="${prefix}_leg">
@@ -141,5 +149,5 @@
       <child link="${prefix}_leg"/>
       <dynamics damping="${JOINT_DAMPING}" friction="${JOINT_FRICTION}"/>
-      <limit effort="30" velocity="1.0" lower="-${GIRDLE_FLEXION_LIMIT}" upper="${GIRDLE_FLEXION_LIMIT}" />
+      <limit effort="${JOINT_MAX_EFFORT}" velocity="${JOINT_MAX_SPEED}" lower="-${GIRDLE_FLEXION_LIMIT}" upper="${GIRDLE_FLEXION_LIMIT}" />
     </joint>
   </xacro:macro>
@@ -155,5 +163,5 @@
    <inertial>
      <origin xyz="0 0 0" rpy="0 0 0"/>
-     <mass value="${BODY_SPHERE_MASS}"/>
+     <mass value="${2*BODY_SPHERE_MASS}"/>
      <inertia ixx="${2*BODY_SPHERE_INERTIA}"  ixy="0"  ixz="0"
               iyy="${2*(BODY_SPHERE_INERTIA+GIRDLE_LENGTH*GIRDLE_LENGTH*BODY_SPHERE_MASS)}" iyz="0"
@@ -237,5 +245,5 @@
     <child link="spine_connection_1"/>
     <dynamics damping="${JOINT_DAMPING}" friction="${JOINT_FRICTION}"/>
-    <limit effort="30" velocity="1.0" lower="-${SPINE_LATERAL_BENDING_LIMIT}" upper="${SPINE_LATERAL_BENDING_LIMIT}" />
+    <limit effort="${JOINT_MAX_EFFORT}" velocity="${JOINT_MAX_SPEED}" lower="-${SPINE_LATERAL_BENDING_LIMIT}" upper="${SPINE_LATERAL_BENDING_LIMIT}" />
   </joint>
   <joint name="spine_dorsal_joint_1" type="revolute">
@@ -245,5 +253,5 @@
     <child link="spine_link_1"/>
     <dynamics damping="${JOINT_DAMPING}" friction="${JOINT_FRICTION}"/>
-    <limit effort="30" velocity="1.0" lower="-${SPINE_DORSAL_BENDING_LIMIT}" upper="${SPINE_DORSAL_BENDING_LIMIT}" />
+    <limit effort="${JOINT_MAX_EFFORT}" velocity="${JOINT_MAX_SPEED}" lower="-${SPINE_DORSAL_BENDING_LIMIT}" upper="${SPINE_DORSAL_BENDING_LIMIT}" />
   </joint>
   <xacro:spine_segments_loop segments_qty="${SPINE_SEGMENTS_NUMBER}"/>

File: crawler_mass_distribution.urdf (robot description, URDF)
Before this commit: robot crawler, 15 links, 14 joints
Links:
- link girdle: mass 0.0008 -> 0.000794
- link spine_link_1: mass 0.0004 -> 0.0006294
- link spine_link_2: mass 0.0004 -> 0.0005857
- link spine_link_3: mass 0.0004 -> 0.0004432
- link spine_link_4: mass 0.0004 -> 0.0002397
- link spine_link_5: mass 0.0004 -> 0.000065
Joints:
- joint left_girdle_flection_joint: limit lower=-0.523598333333 upper=0.523598333333 effort=50.0 velocity=50.0 -> lower=-0.01 upper=0.01 effort=50.0 velocity=50.0
- joint right_girdle_flection_joint: limit lower=-0.523598333333 upper=0.523598333333 effort=50.0 velocity=50.0 -> lower=-0.01 upper=0.01 effort=50.0 velocity=50.0

File: crawler_mass_distribution_long_girdle_bad.urdf (robot description, URDF)
Before this commit: robot crawler, 15 links, 14 joints
Links:
- link girdle: mass 0.0008 -> 0.000794; geometry collision sphere radius=0.00475; collision sphere radius=0.00475
- link spine_link_1: mass 0.0004 -> 0.0006294; geometry collision sphere radius=0.00475; visual box size=0.0108571428571 0.000542857142857 0.000542857142857
- link spine_link_2: mass 0.0004 -> 0.0005857; geometry collision sphere radius=0.00475; visual box size=0.0108571428571 0.000542857142857 0.000542857142857
- link spine_link_3: mass 0.0004 -> 0.0004432; geometry collision sphere radius=0.00475; visual box size=0.0108571428571 0.000542857142857 0.000542857142857
- link spine_link_4: mass 0.0004 -> 0.0002397; geometry collision sphere radius=0.00475; visual box size=0.0108571428571 0.000542857142857 0.000542857142857
- link spine_link_5: mass 0.0004 -> 0.000065; geometry collision sphere radius=0.00475; visual box size=0.0108571428571 0.000542857142857 0.000542857142857
Joints:
- joint left_girdle_abduction_joint: limit lower=-1.570795 upper=1.570795 effort=50.0 velocity=50.0 -> lower=-1.570795 upper=1.570795 effort=30 velocity=1.0
- joint left_girdle_flection_joint: limit lower=-0.523598333333 upper=0.523598333333 effort=50.0 velocity=50.0 -> lower=-0.01 upper=0.01 effort=30 velocity=1.0
- joint right_girdle_abduction_joint: limit lower=-1.570795 upper=1.570795 effort=50.0 velocity=50.0 -> lower=-1.570795 upper=1.570795 effort=30 velocity=1.0
- joint right_girdle_flection_joint: limit lower=-0.523598333333 upper=0.523598333333 effort=50.0 velocity=50.0 -> lower=-0.01 upper=0.01 effort=30 velocity=1.0
- joint spine_dorsal_joint_1: limit lower=-0.39269875 upper=0.39269875 effort=50.0 velocity=50.0 -> lower=-0.39269875 upper=0.39269875 effort=30 velocity=1.0
- joint spine_dorsal_joint_2: limit lower=-0.39269875 upper=0.39269875 effort=50.0 velocity=50.0 -> lower=-0.39269875 upper=0.39269875 effort=30 velocity=1.0
- joint spine_dorsal_joint_3: limit lower=-0.39269875 upper=0.39269875 effort=50.0 velocity=50.0 -> lower=-0.39269875 upper=0.39269875 effort=30 velocity=1.0
- joint spine_dorsal_joint_4: limit lower=-0.39269875 upper=0.39269875 effort=50.0 velocity=50.0 -> lower=-0.39269875 upper=0.39269875 effort=30 velocity=1.0
- joint spine_dorsal_joint_5: limit lower=-0.39269875 upper=0.39269875 effort=50.0 velocity=50.0 -> lower=-0.39269875 upper=0.39269875 effort=30 velocity=1.0
- joint spine_lateral_joint_1: limit lower=-1.570795 upper=1.570795 effort=50.0 velocity=50.0 -> lower=-1.570795 upper=1.570795 effort=30 velocity=1.0; origin xyz=-0.00633333333333 0 0 rpy=0 0 0 -> xyz=-0.0108571428571 0 0 rpy=0 0 0
- joint spine_lateral_joint_2: limit lower=-1.570795 upper=1.570795 effort=50.0 velocity=50.0 -> lower=-1.570795 upper=1.570795 effort=30 velocity=1.0; origin xyz=-0.0126666666667 0 0 rpy=1.570795 0 0 -> xyz=-0.0108571428571 0 0 rpy=1.570795 0 0
- joint spine_lateral_joint_3: limit lower=-1.570795 upper=1.570795 effort=50.0 velocity=50.0 -> lower=-1.570795 upper=1.570795 effort=30 velocity=1.0; origin xyz=-0.0126666666667 0 0 rpy=1.570795 0 0 -> xyz=-0.0108571428571 0 0 rpy=1.570795 0 0
- joint spine_lateral_joint_4: limit lower=-1.570795 upper=1.570795 effort=50.0 velocity=50.0 -> lower=-1.570795 upper=1.570795 effort=30 velocity=1.0; origin xyz=-0.0126666666667 0 0 rpy=1.570795 0 0 -> xyz=-0.0108571428571 0 0 rpy=1.570795 0 0
- joint spine_lateral_joint_5: limit lower=-1.570795 upper=1.570795 effort=50.0 velocity=50.0 -> lower=-1.570795 upper=1.570795 effort=30 velocity=1.0; origin xyz=-0.0126666666667 0 0 rpy=1.570795 0 0 -> xyz=-0.0108571428571 0 0 rpy=1.570795 0 0
