Commit message: Scaled model

File: crawler.urdf.xacro (robot description, xacro)
@@ -6,6 +6,6 @@
   <!--CONSTANTS-->
   <xacro:property name="PI" value="3.14159" />
-  <xacro:property name="BODY_LENGTH" value="0.076"/>
-  <xacro:property name="BODY_MASS" value="0.0028"/>
+  <xacro:property name="BODY_LENGTH" value="0.76"/>
+  <xacro:property name="BODY_MASS" value="2.8"/>
   <xacro:property name="SPINE_SEGMENTS_NUMBER" value="5" />
   <xacro:property name="N_HALF" value="3" />

File: crawler_mass_distribution.urdf (robot description, URDF)
Before this commit: robot crawler, 15 links, 14 joints
Links:
- link girdle: mass 0.000794 -> 0.795; geometry collision sphere radius=0.0475; collision sphere radius=0.0475
- link left_girdle_connection_1: mass 4e-07 -> 0.0004
- link left_leg: mass 4e-05 -> 0.04; geometry collision sphere radius=0.0158333333333; visual box size=0.0808510638298 0.00404255319149 0.00404255319149
- link right_girdle_connection_1: mass 4e-07 -> 0.0004
- link right_leg: mass 4e-05 -> 0.04; geometry collision sphere radius=0.0158333333333; visual box size=0.0808510638298 0.00404255319149 0.00404255319149
- link spine_connection_1: mass 4e-06 -> 0.004
- link spine_connection_2: mass 4e-06 -> 0.004
- link spine_connection_3: mass 4e-06 -> 0.004
- link spine_connection_4: mass 4e-06 -> 0.004
- link spine_connection_5: mass 4e-06 -> 0.004
- link spine_link_1: mass 0.0006294 -> 0.629; geometry collision sphere radius=0.0475; visual box size=0.126666666667 0.00633333333333 0.00633333333333
- link spine_link_2: mass 0.0005857 -> 0.586; geometry collision sphere radius=0.0475; visual box size=0.126666666667 0.00633333333333 0.00633333333333
- link spine_link_3: mass 0.0004432 -> 0.443; geometry collision sphere radius=0.0475; visual box size=0.126666666667 0.00633333333333 0.00633333333333
- link spine_link_4: mass 0.0002397 -> 0.240; geometry collision sphere radius=0.0475; visual box size=0.126666666667 0.00633333333333 0.00633333333333
- link spine_link_5: mass 0.000065 -> 0.065; geometry collision sphere radius=0.0475; visual box size=0.126666666667 0.00633333333333 0.00633333333333
Joints:
- joint left_girdle_abduction_joint: origin xyz=0 0.00542857142857 0 rpy=0 0 1.570795 -> xyz=0 0.0542857142857 0 rpy=0 0 1.570795
- joint left_girdle_flection_joint: limit lower=-0.01 upper=0.01 effort=50.0 velocity=50.0 -> lower=-0.523598333333 upper=0.523598333333 effort=50.0 velocity=50.0
- joint right_girdle_abduction_joint: origin xyz=0 -0.00542857142857 0 rpy=0 0 -1.570795 -> xyz=0 -0.0542857142857 0 rpy=0 0 -1.570795
- joint right_girdle_flection_joint: limit lower=-0.01 upper=0.01 effort=50.0 velocity=50.0 -> lower=-0.523598333333 upper=0.523598333333 effort=50.0 velocity=50.0
- joint spine_lateral_joint_1: origin xyz=-0.00633333333333 0 0 rpy=0 0 0 -> xyz=-0.0633333333333 0 0 rpy=0 0 0
- joint spine_lateral_joint_2: origin xyz=-0.0126666666667 0 0 rpy=1.570795 0 0 -> xyz=-0.126666666667 0 0 rpy=1.570795 0 0
- joint spine_lateral_joint_3: origin xyz=-0.0126666666667 0 0 rpy=1.570795 0 0 -> xyz=-0.126666666667 0 0 rpy=1.570795 0 0
- joint spine_lateral_joint_4: origin xyz=-0.0126666666667 0 0 rpy=1.570795 0 0 -> xyz=-0.126666666667 0 0 rpy=1.570795 0 0
- joint spine_lateral_joint_5: origin xyz=-0.0126666666667 0 0 rpy=1.570795 0 0 -> xyz=-0.126666666667 0 0 rpy=1.570795 0 0

File: small mass/crawler.urdf (robot description, URDF)
Before this commit: robot crawler, 15 links, 14 joints
Links:
- link girdle: mass 0.8 -> 0.0008; geometry collision sphere radius=0.00475; collision sphere radius=0.00475
- link left_girdle_connection_1: mass 0.0004 -> 4e-07
- link left_leg: mass 0.04 -> 4e-05; geometry collision sphere radius=0.00158333333333; visual box size=0.00808510638298 0.000404255319149 0.000404255319149
- link right_girdle_connection_1: mass 0.0004 -> 4e-07
- link right_leg: mass 0.04 -> 4e-05; geometry collision sphere radius=0.00158333333333; visual box size=0.00808510638298 0.000404255319149 0.000404255319149
- link spine_connection_1: mass 0.004 -> 4e-06
- link spine_connection_2: mass 0.004 -> 4e-06
- link spine_connection_3: mass 0.004 -> 4e-06
- link spine_connection_4: mass 0.004 -> 4e-06
- link spine_connection_5: mass 0.004 -> 4e-06
- link spine_link_1: mass 0.4 -> 0.0004; geometry collision sphere radius=0.00475; visual box size=0.0126666666667 0.000633333333333 0.000633333333333
- link spine_link_2: mass 0.4 -> 0.0004; geometry collision sphere radius=0.00475; visual box size=0.0126666666667 0.000633333333333 0.000633333333333
- link spine_link_3: mass 0.4 -> 0.0004; geometry collision sphere radius=0.00475; visual box size=0.0126666666667 0.000633333333333 0.000633333333333
- link spine_link_4: mass 0.4 -> 0.0004; geometry collision sphere radius=0.00475; visual box size=0.0126666666667 0.000633333333333 0.000633333333333
- link spine_link_5: mass 0.4 -> 0.0004; geometry collision sphere radius=0.00475; visual box size=0.0126666666667 0.000633333333333 0.000633333333333
Joints:
- joint left_girdle_abduction_joint: origin xyz=0 0.0542857142857 0 rpy=0 0 1.570795 -> xyz=0 0.00542857142857 0 rpy=0 0 1.570795
- joint right_girdle_abduction_joint: origin xyz=0 -0.0542857142857 0 rpy=0 0 -1.570795 -> xyz=0 -0.00542857142857 0 rpy=0 0 -1.570795
- joint spine_lateral_joint_1: origin xyz=-0.0633333333333 0 0 rpy=0 0 0 -> xyz=-0.00633333333333 0 0 rpy=0 0 0
- joint spine_lateral_joint_2: origin xyz=-0.126666666667 0 0 rpy=1.570795 0 0 -> xyz=-0.0126666666667 0 0 rpy=1.570795 0 0
- joint spine_lateral_joint_3: origin xyz=-0.126666666667 0 0 rpy=1.570795 0 0 -> xyz=-0.0126666666667 0 0 rpy=1.570795 0 0
- joint spine_lateral_joint_4: origin xyz=-0.126666666667 0 0 rpy=1.570795 0 0 -> xyz=-0.0126666666667 0 0 rpy=1.570795 0 0
- joint spine_lateral_joint_5: origin xyz=-0.126666666667 0 0 rpy=1.570795 0 0 -> xyz=-0.0126666666667 0 0 rpy=1.570795 0 0

File: small mass/crawler_mass_distribution.urdf (robot description, URDF)
Before this commit: robot crawler, 15 links, 14 joints
Links:
- link girdle: mass 0.8 -> 0.000794; geometry collision sphere radius=0.00475; collision sphere radius=0.00475
- link left_girdle_connection_1: mass 0.0004 -> 4e-07
- link left_leg: mass 0.04 -> 4e-05; geometry collision sphere radius=0.00158333333333; visual box size=0.00808510638298 0.000404255319149 0.000404255319149
- link right_girdle_connection_1: mass 0.0004 -> 4e-07
- link right_leg: mass 0.04 -> 4e-05; geometry collision sphere radius=0.00158333333333; visual box size=0.00808510638298 0.000404255319149 0.000404255319149
- link spine_connection_1: mass 0.004 -> 4e-06
- link spine_connection_2: mass 0.004 -> 4e-06
- link spine_connection_3: mass 0.004 -> 4e-06
- link spine_connection_4: mass 0.004 -> 4e-06
- link spine_connection_5: mass 0.004 -> 4e-06
- link spine_link_1: mass 0.4 -> 0.0006294; geometry collision sphere radius=0.00475; visual box size=0.0126666666667 0.000633333333333 0.000633333333333
- link spine_link_2: mass 0.4 -> 0.0005857; geometry collision sphere radius=0.00475; visual box size=0.0126666666667 0.000633333333333 0.000633333333333
- link spine_link_3: mass 0.4 -> 0.0004432; geometry collision sphere radius=0.00475; visual box size=0.0126666666667 0.000633333333333 0.000633333333333
- link spine_link_4: mass 0.4 -> 0.0002397; geometry collision sphere radius=0.00475; visual box size=0.0126666666667 0.000633333333333 0.000633333333333
- link spine_link_5: mass 0.4 -> 0.000065; geometry collision sphere radius=0.00475; visual box size=0.0126666666667 0.000633333333333 0.000633333333333
Joints:
- joint left_girdle_abduction_joint: origin xyz=0 0.0542857142857 0 rpy=0 0 1.570795 -> xyz=0 0.00542857142857 0 rpy=0 0 1.570795
- joint left_girdle_flection_joint: limit lower=-0.523598333333 upper=0.523598333333 effort=50.0 velocity=50.0 -> lower=-0.01 upper=0.01 effort=50.0 velocity=50.0
- joint right_girdle_abduction_joint: origin xyz=0 -0.0542857142857 0 rpy=0 0 -1.570795 -> xyz=0 -0.00542857142857 0 rpy=0 0 -1.570795
- joint right_girdle_flection_joint: limit lower=-0.523598333333 upper=0.523598333333 effort=50.0 velocity=50.0 -> lower=-0.01 upper=0.01 effort=50.0 velocity=50.0
- joint spine_lateral_joint_1: origin xyz=-0.0633333333333 0 0 rpy=0 0 0 -> xyz=-0.00633333333333 0 0 rpy=0 0 0
- joint spine_lateral_joint_2: origin xyz=-0.126666666667 0 0 rpy=1.570795 0 0 -> xyz=-0.0126666666667 0 0 rpy=1.570795 0 0
- joint spine_lateral_joint_3: origin xyz=-0.126666666667 0 0 rpy=1.570795 0 0 -> xyz=-0.0126666666667 0 0 rpy=1.570795 0 0
- joint spine_lateral_joint_4: origin xyz=-0.126666666667 0 0 rpy=1.570795 0 0 -> xyz=-0.0126666666667 0 0 rpy=1.570795 0 0
- joint spine_lateral_joint_5: origin xyz=-0.126666666667 0 0 rpy=1.570795 0 0 -> xyz=-0.0126666666667 0 0 rpy=1.570795 0 0
